File: Schematics/AutoSketch/AutoSketch.kicad_sch (KiCad schematic)
At the start: 0 parts

Commit message: EngPrj3
Schematics
Other:
- sheet Interface ports: added Button, OLED-SCL, OLED-SDA, Toggle, Trim; removed Button-Set, Toggle-Set, Trim-Set
- sheet Limit Switches ports: added LimF, LimR; removed none
- sheet MCU ports: added Button, LimF, LimR, OLED-SCL, OLED-SDA, Toggle, Trim; removed Button-Set, Toggle-Set, Trim-Set
- company: (none) -> Fergus Page
- title: (none) -> Top Level System Diagram
Changed lines of the file:
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@@
 	(generator_version "9.0")
 	(paper "A4")
+	(title_block
+		(title "Top Level System Diagram")
+		(date "2025-11-05")
+		(rev "1.0")
+		(company "Fergus Page")
+	)
 	(wire
 		(pts
@@
 	(wire
 		(pts
+			(xy 177.8 87.63) (xy 223.52 87.63)
+		)
+		(stroke
+			(width 0)
+			(type default)
+		)
+	)
+	(wire
+		(pts
 			(xy 177.8 130.81) (xy 223.52 130.81)
 		)
@@
 	(wire
 		(pts
+			(xy 177.8 85.09) (xy 223.52 85.09)
+		)
+		(stroke
+			(width 0)
+			(type default)
+		)
+	)
+	(wire
+		(pts
 			(xy 177.8 29.21) (xy 223.52 29.21)
 		)
@@
 	(wire
 		(pts
+			(xy 73.66 118.11) (xy 123.19 118.11)
+		)
+		(stroke
+			(width 0)
+			(type default)
+		)
+	)
+	(wire
+		(pts
 			(xy 177.8 45.72) (xy 223.52 45.72)
 		)
@@
 	(wire
 		(pts
+			(xy 73.66 120.65) (xy 123.19 120.65)
+		)
+		(stroke
+			(width 0)
+			(type default)
+		)
+	)
+	(wire
+		(pts
 			(xy 177.8 133.35) (xy 223.52 133.35)
 		)
@@
 		(pts
 			(xy 73.66 87.63) (xy 123.19 87.63)
+		)
+		(stroke
+			(width 0)
+			(type default)
+		)
+	)
+	(wire
+		(pts
+			(xy 73.025 139.7) (xy 123.19 139.7)
 		)
 		(stroke
@@
 			(project "AutoSketch"
 				(path "/da5a1e6a-2605-436b-a30c-1027586d5c0a"
-					(page "6")
+					(page "10")
 				)
 			)
@@
 	)
 	(sheet
-		(at 224.155 147.32)
+		(at 19.685 131.445)
 		(size 53.34 15.24)
 		(exclude_from_sim no)
@@
 		)
 		(property "Sheetname" "Vibrating Motor"
-			(at 224.155 146.6084 0)
+			(at 19.685 130.7334 0)
 			(effects
 				(font
@@
 		)
 		(property "Sheetfile" "vibe.kicad_sch"
-			(at 224.155 163.1446 0)
+			(at 19.685 147.2696 0)
 			(effects
 				(font
@@
 		)
 		(property "Field2" ""
-			(at 224.155 147.32 0)
+			(at 19.685 131.445 0)
 			(effects
 				(font
@@
 		)
 		(pin "Vibe" input
-			(at 224.155 151.13 180)
-			(effects
-				(font
-					(size 1.27 1.27)
-				)
-				(justify left)
+			(at 73.025 139.7 0)
+			(effects
+				(font
+					(size 1.27 1.27)
+				)
+				(justify right)
 			)
 		)
@@
 			)
 		)
-		(pin "Button-Set" output
+		(pin "OLED-SCL" input
+			(at 73.66 118.11 0)
+			(effects
+				(font
+					(size 1.27 1.27)
+				)
+				(justify right)
+			)
+		)
+		(pin "OLED-SDA" bidirectional
+			(at 73.66 120.65 0)
+			(effects
+				(font
+					(size 1.27 1.27)
+				)
+				(justify right)
+			)
+		)
+		(pin "Button" output
+			(at 73.66 110.49 0)
+			(effects
+				(font
+					(size 1.27 1.27)
+				)
+				(justify right)
+			)
+		)
+		(pin "Toggle" output
 			(at 73.66 113.03 0)
 			(effects
@@
 			)
 		)
-		(pin "Toggle-Set" output
-			(at 73.66 110.49 0)
-			(effects
-				(font
-					(size 1.27 1.27)
-				)
-				(justify right)
-			)
-		)
-		(pin "Trim-Set" output
+		(pin "Trim" output
 			(at 73.66 115.57 0)
 			(effects
@@
 			(project "AutoSketch"
 				(path "/da5a1e6a-2605-436b-a30c-1027586d5c0a"
-					(page "4")
+					(page "7")
 				)
 			)
@@
 			(project "AutoSketch"
 				(path "/da5a1e6a-2605-436b-a30c-1027586d5c0a"
-					(page "3")
+					(page "2")
 				)
 			)
@@
 	(sheet
 		(at 123.19 20.32)
-		(size 54.61 142.24)
+		(size 54.61 130.81)
 		(exclude_from_sim no)
 		(in_bom yes)
@@
 		)
 		(property "Sheetfile" "mcu.kicad_sch"
-			(at 123.19 163.1446 0)
+			(at 123.19 151.7146 0)
 			(effects
 				(font
@@
 			)
 		)
-		(pin "Button-Set" input
-			(at 123.19 113.03 180)
-			(effects
-				(font
-					(size 1.27 1.27)
-				)
-				(justify left)
-			)
-		)
-		(pin "Toggle-Set" input
-			(at 123.19 110.49 180)
-			(effects
-				(font
-					(size 1.27 1.27)
-				)
-				(justify left)
-			)
-		)
-		(pin "Trim-Set" input
-			(at 123.19 115.57 180)
-			(effects
-				(font
-					(size 1.27 1.27)
-				)
-				(justify left)
-			)
-		)
 		(pin "Wireless-CE" output
 			(at 123.19 80.01 180)
@@
 		)
 		(pin "Vibe" output
-			(at 177.8 151.13 0)
-			(effects
-				(font
-					(size 1.27 1.27)
-				)
-				(justify right)
+			(at 123.19 139.7 180)
+			(effects
+				(font
+					(size 1.27 1.27)
+				)
+				(justify left)
+			)
+		)
+		(pin "LimF" input
+			(at 177.8 85.09 0)
+			(effects
+				(font
+					(size 1.27 1.27)
+				)
+				(justify right)
+			)
+		)
+		(pin "LimR" input
+			(at 177.8 87.63 0)
+			(effects
+				(font
+					(size 1.27 1.27)
+				)
+				(justify right)
+			)
+		)
+		(pin "OLED-SCL" output
+			(at 123.19 118.11 180)
+			(effects
+				(font
+					(size 1.27 1.27)
+				)
+				(justify left)
+			)
+		)
+		(pin "OLED-SDA" bidirectional
+			(at 123.19 120.65 180)
+			(effects
+				(font
+					(size 1.27 1.27)
+				)
+				(justify left)
+			)
+		)
+		(pin "Button" input
+			(at 123.19 110.49 180)
+			(effects
+				(font
+					(size 1.27 1.27)
+				)
+				(justify left)
+			)
+		)
+		(pin "Toggle" input
+			(at 123.19 113.03 180)
+			(effects
+				(font
+					(size 1.27 1.27)
+				)
+				(justify left)
+			)
+		)
+		(pin "Trim" input
+			(at 123.19 115.57 180)
+			(effects
+				(font
+					(size 1.27 1.27)
+				)
+				(justify left)
 			)
 		)
@@
 			(project "AutoSketch"
 				(path "/da5a1e6a-2605-436b-a30c-1027586d5c0a"
-					(page "2")
+					(page "4")
 				)
 			)
@@
 			)
 		)
+		(pin "LimF" output
+			(at 223.52 85.09 180)
+			(effects
+				(font
+					(size 1.27 1.27)
+				)
+				(justify left)
+			)
+		)
+		(pin "LimR" output
+			(at 223.52 87.63 180)
+			(effects
+				(font
+					(size 1.27 1.27)
+				)
+				(justify left)
+			)
+		)
 		(instances
 			(project "AutoSketch"
@@
 			(project "AutoSketch"
 				(path "/da5a1e6a-2605-436b-a30c-1027586d5c0a"
-					(page "10")
+					(page "3")
 				)
 			)
@@
 			(project "AutoSketch"
 				(path "/da5a1e6a-2605-436b-a30c-1027586d5c0a"
-					(page "7")
+					(page "5")
 				)
 			)
@@
 			(project "AutoSketch"
 				(path "/da5a1e6a-2605-436b-a30c-1027586d5c0a"
-					(page "5")
-				)
-			)
+					(page "6")
+				)
+			)
