File: Schematics/AutoSketch/dcm.kicad_sch (KiCad schematic)
At the start: 3 parts, among them M1 Motor_DC, U2 L293D

Commit message: EngPrj3
Schematics
Parts:
- added D2, D3: LED, symbol Device:LED
- added R15, R16, R17, R18: 10k, symbol Device:R
- added R21, R22: 1k, symbol Device:R
- added U4: TL084, symbol Amplifier_Operational:TL084
Connections:
- net GND: now also D2.1 (K), D3.1 (K)
- net at M1.1 (+), U2.3 (1Y): now also U2.14 (4Y), R15.1, U4.12 (+); no longer U2.11 (3Y)
- net at M1.2 (-), U2.6 (2Y): now also U2.11 (3Y), R18.2, U4.10 (+); no longer U2.14 (4Y)
- new net: R17.1, R22.2, U4.14
- new net: R17.2, R18.1, U4.13 (-)
- new net: R15.2, R16.1, U4.9 (-)
- new net: R16.2, R21.2, U4.8
- new net: D3.2 (A), R22.1
- new net: D2.2 (A), R21.1
Other:
- company: (none) -> Fergus Page
- title: (none) -> DC Motor, Driver, and Indicators
- moved on the sheet: C1
