File: Schematics/AutoSketch/encoder.kicad_sch (KiCad schematic)
At the start: 11 parts, among them U4 TL084

Commit message: EngPrj3
Schematics
Parts:
- removed R15, R16, R17, R18: 10k, symbol Device:R
- removed unit 3 of U4
- removed unit 4 of U4
Other:
- company: (none) -> Fergus Page
- title: (none) -> Encoders and Conditioning
