File: Schematics/AutoSketch/interface.kicad_sch (KiCad schematic)
At the start: 4 parts, among them SW1 Toggle, SW2 Button

Commit message: EngPrj3
Schematics
Parts:
- added U6: SSD1306, symbol GrandOleLirbrarey:Generic_I2C
Connections:
- net GND: now also U6.2 (GND)
- net R3V3: now also U6.1 (Vcc)
- net Button-Set renamed Button
- net Toggle-Set renamed Toggle
- net Trim-Set renamed Trim
- new net OLED-SCL: U6.3 (SCL)
- new net OLED-SDA: U6.4 (SDA)
Other:
- note added: "OLED Display"
- company: (none) -> Fergus Page
- title: (none) -> Hardware User Interface
Changed lines of the file:
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@@
 	(generator_version "9.0")
 	(paper "A4")
+	(title_block
+		(title "Hardware User Interface")
+		(date "2025-11-05")
+		(rev "1.0")
+		(company "Fergus Page")
+	)
+	(text "OLED Display"
+		(exclude_from_sim no)
+		(at 195.072 48.514 0)
+		(effects
+			(font
+				(size 1.27 1.27)
+			)
+		)
+	)
 	(junction
 		(at 76.2 52.07)
@@
 	)
 	(junction
+		(at 142.24 85.09)
+		(diameter 0)
+		(color 0 0 0 0)
+	)
+	(junction
 		(at 96.52 85.09)
+		(diameter 0)
+		(color 0 0 0 0)
+	)
+	(junction
+		(at 142.24 52.07)
 		(diameter 0)
 		(color 0 0 0 0)
@@
 	(wire
 		(pts
+			(xy 195.58 52.07) (xy 142.24 52.07)
+		)
+		(stroke
+			(width 0)
+			(type default)
+		)
+	)
+	(wire
+		(pts
 			(xy 146.05 78.74) (xy 153.67 78.74)
 		)
@@
 	(wire
 		(pts
+			(xy 195.58 82.55) (xy 195.58 85.09)
+		)
+		(stroke
+			(width 0)
+			(type default)
+		)
+	)
+	(wire
+		(pts
 			(xy 105.41 60.96) (xy 105.41 72.39)
 		)
@@
 	(wire
 		(pts
+			(xy 195.58 57.15) (xy 195.58 52.07)
+		)
+		(stroke
+			(width 0)
+			(type default)
+		)
+	)
+	(wire
+		(pts
 			(xy 105.41 83.82) (xy 105.41 85.09)
 		)
@@
 	(wire
 		(pts
+			(xy 180.34 69.85) (xy 184.15 69.85)
+		)
+		(stroke
+			(width 0)
+			(type default)
+		)
+	)
+	(wire
+		(pts
 			(xy 81.28 53.34) (xy 81.28 54.61)
 		)
@@
 		(pts
 			(xy 105.41 52.07) (xy 142.24 52.07)
+		)
+		(stroke
+			(width 0)
+			(type default)
+		)
+	)
+	(wire
+		(pts
+			(xy 180.34 72.39) (xy 184.15 72.39)
+		)
+		(stroke
+			(width 0)
+			(type default)
+		)
+	)
+	(wire
+		(pts
+			(xy 195.58 85.09) (xy 142.24 85.09)
 		)
 		(stroke
@@
 		)
 	)
-	(hierarchical_label "Toggle-Set"
+	(hierarchical_label "Toggle"
 		(shape output)
 		(at 153.67 66.04 0)
@@
 		)
 	)
-	(hierarchical_label "Button-Set"
+	(hierarchical_label "Button"
 		(shape output)
 		(at 153.67 72.39 0)
@@
 		)
 	)
-	(hierarchical_label "Trim-Set"
+	(hierarchical_label "OLED-SCL"
+		(shape input)
+		(at 180.34 69.85 180)
+		(effects
+			(font
+				(size 1.27 1.27)
+			)
+			(justify right)
+		)
+	)
+	(hierarchical_label "OLED-SDA"
+		(shape bidirectional)
+		(at 180.34 72.39 180)
+		(effects
+			(font
+				(size 1.27 1.27)
+			)
+			(justify right)
+		)
+	)
+	(hierarchical_label "Trim"
 		(shape output)
 		(at 153.67 78.74 0)
@@
 					(unit 1)
 				)
+			)
+		)
+	)
+	(symbol
+		(lib_id "GrandOleLirbrarey:Generic_I2C")
+		(at 189.23 62.23 0)
+		(unit 1)
+		(exclude_from_sim no)
+		(in_bom no)
+		(on_board no)
+		(dnp no)
+		(property "Reference" "U6"
+			(at 194.818 69.342 0)
+			(effects
+				(font
+					(size 1.27 1.27)
+				)
+				(justify left)
+			)
+		)
+		(property "Value" "SSD1306"
+			(at 194.818 71.374 0)
+			(effects
+				(font
+					(size 1.27 1.27)
+				)
+				(justify left)
+			)
+		)
+		(property "Footprint" ""
+			(at 189.23 62.23 0)
+			(effects
+				(font
+					(size 1.27 1.27)
+				)
+				(hide yes)
+			)
+		)
+		(property "Datasheet" ""
+			(at 189.23 62.23 0)
+			(effects
+				(font
+					(size 1.27 1.27)
+				)
+				(hide yes)
+			)
+		)
+		(property "Description" ""
+			(at 189.23 62.23 0)
+			(effects
+				(font
+					(size 1.27 1.27)
+				)
+				(hide yes)
+			)
+		)
+		(pin "4"
+		)
+		(pin "2"
+		)
+		(pin "3"
+		)
+		(pin "1"
+		)
+		(instances
+			(project ""
+				(path "/da5a1e6a-2605-436b-a30c-1027586d5c0a/631ff66c-e0f1-44f6-b7c1-b700e9b00805"
+					(reference "U6")
+					(unit 1)
+				)
