File: Schematics/AutoSketch/limit.kicad_sch (KiCad schematic)
At the start: 0 parts

Commit message: EngPrj3
Schematics
Parts:
- added R19, R20: 10k, symbol Device:R
- added SW3, SW4: Button, symbol Switch:SW_SPST
Connections:
- new net GND: SW3.2 (B), SW4.2 (B)
- new net LimF: R19.2, SW3.1 (A)
- new net LimR: R20.2, SW4.1 (A)
- new net R5V: R19.1, R20.1
Other:
- company: (none) -> Fergus Page
- title: (none) -> Limit Switches
