File: Schematics/AutoSketch/mcu.kicad_sch (KiCad schematic)
At the start: 5 parts, among them J1 CN7, J2 CN10

Commit message: EngPrj3
Schematics
Other:
- company: (none) -> Fergus Page
Changed lines of the file:
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@@
 	(generator_version "9.0")
 	(paper "A4")
+	(title_block
+		(date "2025-11-05")
+		(rev "1.0")
+		(company "Fergus Page")
+	)
 	(text "Mechanical\n"
 		(exclude_from_sim no)
@@
 	(global_label "R3V3"
 		(shape output)
-		(at 201.93 27.94 180)
+		(at 139.7 33.02 180)
 		(fields_autoplaced yes)
 		(effects
@@
 		)
 		(property "Intersheetrefs" "${INTERSHEET_REFS}"
-			(at 194.1672 27.94 0)
+			(at 131.9372 33.02 0)
 			(effects
 				(font
@@
 	(hierarchical_label "Y-EN~"
 		(shape output)
-		(at 109.22 137.16 180)
-		(effects
-			(font
-				(size 1.27 1.27)
-			)
-			(justify right)
+		(at 199.39 52.705 0)
+		(effects
+			(font
+				(size 1.27 1.27)
+			)
+			(justify left)
 		)
 	)
 	(hierarchical_label "X-Reset~"
 		(shape output)
-		(at 93.98 129.54 180)
-		(effects
-			(font
-				(size 1.27 1.27)
-			)
-			(justify right)
-		)
-	)
-	(hierarchical_label "Toggle-Set"
-		(shape input)
-		(at 30.48 125.73 0)
+		(at 59.69 24.13 180)
+		(effects
+			(font
+				(size 1.27 1.27)
+			)
+			(justify right)
+		)
+	)
+	(hierarchical_label "Toggle"
+		(shape input)
+		(at 208.28 91.44 0)
+		(effects
+			(font
+				(size 1.27 1.27)
+			)
+			(justify left)
+		)
+	)
+	(hierarchical_label "OLED-SDA"
+		(shape bidirectional)
+		(at 209.55 102.87 0)
 		(effects
 			(font
@@
 	(hierarchical_label "Encoder-B"
 		(shape input)
-		(at 30.48 63.5 0)
-		(effects
-			(font
-				(size 1.27 1.27)
-			)
-			(justify left)
+		(at 99.06 21.59 180)
+		(effects
+			(font
+				(size 1.27 1.27)
+			)
+			(justify right)
 		)
 	)
 	(hierarchical_label "Y-Mode1"
 		(shape output)
-		(at 109.22 147.32 180)
-		(effects
-			(font
-				(size 1.27 1.27)
-			)
-			(justify right)
+		(at 199.39 42.545 0)
+		(effects
+			(font
+				(size 1.27 1.27)
+			)
+			(justify left)
 		)
 	)
 	(hierarchical_label "Y-Dir"
 		(shape output)
-		(at 109.22 142.24 180)
-		(effects
-			(font
-				(size 1.27 1.27)
-			)
-			(justify right)
+		(at 199.39 47.625 0)
+		(effects
+			(font
+				(size 1.27 1.27)
+			)
+			(justify left)
 		)
 	)
 	(hierarchical_label "X-Mode3"
 		(shape output)
-		(at 93.98 152.4 180)
+		(at 59.69 46.99 180)
 		(effects
 			(font
@@
 	(hierarchical_label "Y-Mode2"
 		(shape output)
-		(at 109.22 149.86 180)
-		(effects
-			(font
-				(size 1.27 1.27)
-			)
-			(justify right)
+		(at 199.39 40.005 0)
+		(effects
+			(font
+				(size 1.27 1.27)
+			)
+			(justify left)
 		)
 	)
 	(hierarchical_label "DC-Set"
 		(shape output)
-		(at 40.64 83.82 180)
+		(at 57.15 83.82 180)
 		(effects
 			(font
@@
 	(hierarchical_label "DC-Feedback"
 		(shape output)
-		(at 40.64 87.63 180)
+		(at 57.15 87.63 180)
 		(effects
 			(font
@@
 	(hierarchical_label "Y-Step"
 		(shape output)
-		(at 109.22 139.7 180)
+		(at 199.39 50.165 0)
+		(effects
+			(font
+				(size 1.27 1.27)
+			)
+			(justify left)
+		)
+	)
+	(hierarchical_label "LimF"
+		(shape input)
+		(at 99.06 33.02 180)
 		(effects
 			(font
@@
 	(hierarchical_label "Wireless-SCK"
 		(shape output)
-		(at 41.91 102.87 180)
-		(effects
-			(font
-				(size 1.27 1.27)
-			)
-			(justify right)
+		(at 208.28 78.74 0)
+		(effects
+			(font
+				(size 1.27 1.27)
+			)
+			(justify left)
 		)
 	)
 	(hierarchical_label "DC-Direction"
 		(shape output)
-		(at 40.64 73.66 180)
+		(at 57.15 73.66 180)
 		(effects
 			(font
@@
 	(hierarchical_label "DC-Direction~"
 		(shape output)
-		(at 40.64 78.74 180)
+		(at 57.15 78.74 180)
 		(effects
 			(font
@@
 	(hierarchical_label "Y-Reset~"
 		(shape output)
-		(at 109.22 129.54 180)
-		(effects
-			(font
-				(size 1.27 1.27)
-			)
-			(justify right)
+		(at 199.39 60.325 0)
+		(effects
+			(font
+				(size 1.27 1.27)
+			)
+			(justify left)
 		)
 	)
 	(hierarchical_label "Wireless-MOSI"
 		(shape output)
-		(at 41.91 97.79 180)
-		(effects
-			(font
-				(size 1.27 1.27)
-			)
-			(justify right)
+		(at 208.28 83.82 0)
+		(effects
+			(font
+				(size 1.27 1.27)
+			)
+			(justify left)
 		)
 	)
 	(hierarchical_label "X-Mode1"
 		(shape output)
-		(at 93.98 147.32 180)
+		(at 59.69 41.91 180)
 		(effects
 			(font
@@
 	(hierarchical_label "X-Sleep~"
 		(shape output)
-		(at 93.98 132.08 180)
+		(at 59.69 26.67 180)
 		(effects
 			(font
@@
 	(hierarchical_label "Wireless-MISO"
 		(shape input)
-		(at 41.91 100.33 180)
-		(effects
-			(font
-				(size 1.27 1.27)
-			)
-			(justify right)
+		(at 208.28 81.28 0)
+		(effects
+			(font
+				(size 1.27 1.27)
+			)
+			(justify left)
 		)
 	)
 	(hierarchical_label "X-Step"
 		(shape output)
-		(at 93.98 139.7 180)
+		(at 59.69 34.29 180)
 		(effects
 			(font
@@
 	(hierarchical_label "Y-Mode3"
 		(shape output)
-		(at 109.22 152.4 180)
-		(effects
-			(font
-				(size 1.27 1.27)
-			)
-			(justify right)
+		(at 199.39 37.465 0)
+		(effects
+			(font
+				(size 1.27 1.27)
+			)
+			(justify left)
 		)
 	)
 	(hierarchical_label "Vibe"
 		(shape output)
-		(at 36.83 148.59 180)
-		(effects
-			(font
-				(size 1.27 1.27)
-			)
-			(justify right)
-		)
-	)
-	(hierarchical_label "Button-Set"
-		(shape input)
-		(at 30.48 132.08 0)
+		(at 99.06 35.56 180)
+		(effects
+			(font
+				(size 1.27 1.27)
+			)
+			(justify right)
+		)
+	)
+	(hierarchical_label "Button"
+		(shape input)
+		(at 208.28 93.98 0)
 		(effects
 			(font
@@
 	(hierarchical_label "Wireless-CE"
 		(shape output)
-		(at 41.91 110.49 180)
-		(effects
-			(font
-				(size 1.27 1.27)
-			)
-			(justify right)
+		(at 208.28 76.2 0)
+		(effects
+			(font
+				(size 1.27 1.27)
+			)
+			(justify left)
 		)
 	)
 	(hierarchical_label "X-Mode2"
 		(shape output)
-		(at 93.98 149.86 180)
+		(at 59.69 44.45 180)
 		(effects
 			(font
@@
 	(hierarchical_label "X-EN~"
 		(shape output)
-		(at 93.98 137.16 180)
+		(at 59.69 31.75 180)
 		(effects
 			(font
@@
 	(hierarchical_label "Y-Sleep~"
 		(shape output)
-		(at 109.22 132.08 180)
-		(effects
-			(font
-				(size 1.27 1.27)
-			)
-			(justify right)
+		(at 199.39 57.785 0)
+		(effects
+			(font
+				(size 1.27 1.27)
+			)
+			(justify left)
+		)
+	)
+	(hierarchical_label "OLED-SCL"
+		(shape output)
+		(at 209.55 105.41 0)
+		(effects
+			(font
+				(size 1.27 1.27)
+			)
+			(justify left)
 		)
 	)
 	(hierarchical_label "Encoder-A"
 		(shape input)
-		(at 30.48 58.42 0)
-		(effects
-			(font
-				(size 1.27 1.27)
-			)
-			(justify left)
-		)
-	)
-	(hierarchical_label "Trim-Set"
-		(shape input)
-		(at 30.48 138.43 0)
-		(effects
-			(font
-				(size 1.27 1.27)
-			)
-			(justify left)
+		(at 99.06 26.67 180)
+		(effects
+			(font
+				(size 1.27 1.27)
+			)
+			(justify right)
+		)
+	)
+	(hierarchical_label "Trim"
+		(shape input)
+		(at 208.28 96.52 0)
+		(effects
+			(font
+				(size 1.27 1.27)
+			)
+			(justify left)
+		)
+	)
+	(hierarchical_label "LimR"
+		(shape input)
+		(at 99.06 30.48 180)
+		(effects
+			(font
+				(size 1.27 1.27)
+			)
+			(justify right)
 		)
 	)
 	(hierarchical_label "Wireless-IRQ"
 		(shape input)
-		(at 41.91 113.03 180)
-		(effects
-			(font
-				(size 1.27 1.27)
-			)
-			(justify right)
+		(at 208.28 73.66 0)
+		(effects
+			(font
+				(size 1.27 1.27)
+			)
+			(justify left)
 		)
 	)
 	(hierarchical_label "X-Dir"
 		(shape output)
-		(at 93.98 142.24 180)
-		(effects
-			(font
+		(at 59.69 36.83 180)
+		(effects
+			(font
