File: Schematics/AutoSketch/pid.kicad_sch (KiCad schematic)
At the start: 7 parts, among them U3 TL084

Commit message: EngPrj3
Schematics
Other:
- company: (none) -> Fergus Page
- title: (none) -> PID Controller
Changed lines of the file:
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@@
 	(generator_version "9.0")
 	(paper "A4")
+	(title_block
+		(title "PID Controller")
+		(date "2025-11-05")
+		(rev "1.0")
+		(company "Fergus Page")
+	)
 	(junction
 		(at 88.9 87.63)
@@
 	(hierarchical_label "DC-Control"
 		(shape output)
-		(at 194.31 101.6 0)
+		(at 76.2 67.31 0)
 		(effects
 			(font
