File: Schematics/AutoSketch/power.kicad_sch (KiCad schematic)
At the start: 4 parts

Commit message: EngPrj3
Schematics
Other:
- company: (none) -> Fergus Page
- title: (none) -> Power
Changed lines of the file:
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@@
 	(generator_version "9.0")
 	(paper "A4")
+	(title_block
+		(title "Power")
+		(date "2025-11-05")
+		(rev "1.0")
+		(company "Fergus Page")
+	)
 	(junction
 		(at 123.19 57.15)
