File: Schematics/AutoSketch/rpi5.kicad_sch (KiCad schematic)
At the start: 0 parts

Commit message: EngPrj3
Schematics
Parts:
- added J3: Raspberry_Pi_4, symbol Connector:Raspberry_Pi_4
- added J4: Conn_02x05_Odd_Even, symbol Connector_Generic:Conn_02x05_Odd_Even
Connections:
- new net: J3.1 (3V3), J3.17 (3V3)
- new net GND: J3.14 (GND), J3.20 (GND), J3.25 (GND), J3.30 (GND), J3.34 (GND), J3.39 (GND), J3.6 (GND), J3.9 (GND)
- new net R5V: J3.2 (5V), J3.4 (5V)
Other:
- company: (none) -> Fergus Page
- title: (none) -> R Pi 5 10-Pin Wire Interface
