File: Schematics/AutoSketch/sm.kicad_sch (KiCad schematic)
At the start: 4 parts, among them M2 X-Stepper, M3 Y-Stepper

Commit message: EngPrj3
Schematics
Other:
- company: (none) -> Fergus Page
- title: (none) -> Stepper Motor Stylus Control
Changed lines of the file:
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@@
 	(generator_version "9.0")
 	(paper "A4")
+	(title_block
+		(title "Stepper Motor Stylus Control")
+		(date "2025-11-05")
+		(rev "1.0")
+		(company "Fergus Page")
+	)
 	(junction
 		(at 91.44 118.11)
