File: Schematics/AutoSketch/wireless.kicad_sch (KiCad schematic)
At the start: 1 part, among them U1 NRF24L01_Breakout

Commit message: EngPrj3
Schematics
Other:
- company: (none) -> Fergus Page
- title: (none) -> Wireless
Changed lines of the file:
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@@
 	(generator_version "9.0")
 	(paper "A4")
+	(title_block
+		(title "Wireless")
+		(date "2025-11-05")
+		(rev "1.0")
+		(company "Fergus Page")
+	)
 	(junction
 		(at 106.68 102.87)
